Commit message: modified for tars5 sensor kit

File: awsim_sensor_kit_description/urdf/sensor_kit.xacro (robot description, xacro)
@@ -9,5 +9,5 @@
     <xacro:arg name="config_dir" default="$(find awsim_sensor_kit_description)/config"/>
     <xacro:property name="sensor_kit_base_link" default="sensor_kit_base_link"/>
-    <joint name="${sensor_kit_base_link}_joint" type="fixed">
+    <!-- <joint name="${sensor_kit_base_link}_joint" type="fixed">
       <origin rpy="${roll} ${pitch} ${yaw}" xyz="${x} ${y} ${z}"/>
       <parent link="${parent}"/>
@@ -16,19 +16,39 @@
     <link name="${sensor_kit_base_link}">
       <origin rpy="0 0 0" xyz="0 0 0"/>
-    </link>
+    </link> -->
     <!-- sensor -->
     <xacro:property name="calibration" value="${xacro.load_yaml('$(arg config_dir)/sensor_kit_calibration.yaml')}"/>
     <!-- lidar Unity [z,x,y] = [x,y,z] in ROS-->
-    <xacro:VLS-128 parent="base_link" name="velodyne_top" topic="/points_raw" hz="10" samples="220" gpu="$(arg gpu)">
-      <origin
-        xyz="-2.281
-        0
-        1.848"
+    <xacro:VLS-128 parent="base_link" name="velodyne" topic="/points_raw" hz="10" samples="220" gpu="$(arg gpu)">
+      <origin
+        xyz="0.2202
+        0
+        0.6781"
+        rpy="0
+        0
+        4.712"
+      />
+    </xacro:VLS-128>
+    <!-- <xacro:VLS-128 parent="base_link" name="velodyne2" topic="/points_raw2" hz="10" samples="220" gpu="$(arg gpu)">
+      <origin
+        xyz="0.2202
+        0
+        0.6781"
+        rpy="0
+        0
+        4.712"
+      />
+    </xacro:VLS-128> -->
+    <!-- <xacro:VLS-128 parent="base_link" name="zed2i_left_camera_frame" topic="/zed2i/zed_node/point_cloud/cloud_registered" hz="10" samples="220" gpu="$(arg gpu)">
+      <origin
+        xyz="0.2202
+        0
+        0.7381"
         rpy="0
         0
         0"
       />
-    </xacro:VLS-128>
-    <xacro:VLP-16 parent="base_link" name="velodyne_left" topic="/points_raw" hz="10" samples="220" gpu="$(arg gpu)">
+    </xacro:VLS-128> -->
+    <!-- <xacro:VLP-16 parent="base_link" name="velodyne_left" topic="/points_raw" hz="10" samples="220" gpu="$(arg gpu)">
       <origin
         xyz="2.63
@@ -49,5 +69,5 @@
         0"
       />
-    </xacro:VLP-16>
+    </xacro:VLP-16> -->
     <!-- camera -->
     <!-- <xacro:monocular_camera_macro
@@ -66,5 +86,5 @@
       fov="1.3"
     /> -->
-    <xacro:monocular_camera_macro
+    <!-- <xacro:monocular_camera_macro
       name="traffic_light_left_camera/camera"
       parent="base_link"
@@ -80,5 +100,5 @@
       height="400"
       fov="1.3"
-    />
+    /> -->
     <!-- <xacro:monocular_camera_macro
       name="camera0/camera"
@@ -173,10 +193,10 @@
     <!-- gnss -->
     <xacro:imu_macro
-      name="gnss"
-      parent="sensor_kit_base_link"
-      namespace=""
-      x="0"
+      name="gps_link"
+      parent="base_link"
+      namespace=""
+      x="0.2"
       y="0"
-      z="0"
+      z="0.2"
       roll="0"
       pitch="0"
@@ -186,10 +206,10 @@
     <!-- imu -->
     <xacro:imu_macro
-      name="tamagawa/imu"
-      parent="sensor_kit_base_link"
-      namespace=""
-      x="0"
-      y="0"
-      z="0"
+      name="imu"
+      parent="base_link"
+      namespace=""
+      x="0.20479"
+      y="0.13368"
+      z="0.15538"
       roll="0"
       pitch="0"

Commit message: 8 seater buggy changes

File: awsim_sensor_kit_description/urdf/sensor_kit.xacro (robot description, xacro)
@@ -20,24 +20,34 @@
     <xacro:property name="calibration" value="${xacro.load_yaml('$(arg config_dir)/sensor_kit_calibration.yaml')}"/>
     <!-- lidar Unity [z,x,y] = [x,y,z] in ROS-->
-    <xacro:VLS-128 parent="base_link" name="velodyne" topic="/points_raw" hz="10" samples="220" gpu="$(arg gpu)">
-      <origin
-        xyz="0.2202
-        0
-        0.6781"
-        rpy="0
-        0
-        4.712"
+    <xacro:VLS-128 parent="base_link" name="velodyne_top" topic="/points_raw/top" hz="10" samples="220" gpu="$(arg gpu)">
+      <origin
+        xyz="-0.478
+        0.0125
+        1.952"
+        rpy="0
+        0
+        3.141592"
       />
     </xacro:VLS-128>
-    <!-- <xacro:VLS-128 parent="base_link" name="velodyne2" topic="/points_raw2" hz="10" samples="220" gpu="$(arg gpu)">
-      <origin
-        xyz="0.2202
-        0
-        0.6781"
-        rpy="0
-        0
-        4.712"
-      />
-    </xacro:VLS-128> -->
+    <xacro:VLS-128 parent="base_link" name="velodyne_left" topic="/sensing/lidar/left/points_raw" hz="10" samples="220" gpu="$(arg gpu)">
+      <origin
+        xyz="3.105
+          0.535
+          1.226"
+          rpy="0
+          0
+          0.1"
+      />
+    </xacro:VLS-128>
+    <xacro:VLS-128 parent="base_link" name="velodyne_right" topic="/sensing/lidar/right/points_raw" hz="10" samples="220" gpu="$(arg gpu)">
+      <origin
+          xyz="3.105
+          -0.535
+          1.226"
+          rpy="0
+          0
+          0"
+      />
+    </xacro:VLS-128>
     <!-- <xacro:VLS-128 parent="base_link" name="zed2i_left_camera_frame" topic="/zed2i/zed_node/point_cloud/cloud_registered" hz="10" samples="220" gpu="$(arg gpu)">
       <origin
@@ -206,10 +216,10 @@
     <!-- imu -->
     <xacro:imu_macro
-      name="imu"
+      name="zed_imu"
       parent="base_link"
       namespace=""
-      x="0.20479"
-      y="0.13368"
-      z="0.15538"
+      x="3.0"
+      y="0"
+      z="1.0"
       roll="0"
       pitch="0"
